Commit message: refactor: split xacro files

File: twr_description/urdf/twr.urdf.xacro (robot description, xacro)
@@ -1,46 +1,61 @@
 <?xml version="1.0"?>
 <robot name="twr" xmlns:xacro="http://ros.org/wiki/xacro">
+    <xacro:include filename="inertia.macro.xacro"/>
+    <xacro:include filename="colors.xacro"/>
+    <xacro:property name="base_length" value="0.7"/>
     <xacro:property name="base_width" value="0.4"/>
-    <xacro:property name="base_length" value="0.7"/>
-    <xacro:property name="base_height" value="0.05"/>
-    <xacro:macro name="box_inertia" params="m w h d">
-        <inertial>
-            <origin xyz="0.0 0.0 0.0" rpy="${pi/2} 0.0 ${pi/2}"/>
-        <mass value="${m}"/>
-        <inertia
-            ixx="${(m/12) * (h*h + d*d)}" ixy="0.0" ixz="0.0"
-            iyy="${(m/12) * (w*w + d*d)}" iyz="0.0"
-            izz="${(m/12) * (w*w + h*h)}"/>
-        </inertial>
-    </xacro:macro>
-    <link name="dummy_link"/>
-    <joint name="dummy_joint" type="fixed">
-        <parent link="dummy_link"/>
+    <xacro:property name="base_height" value="0.1"/>
+    <xacro:property name="wheel_radius" value="0.2"/>
+    <xacro:property name="wheel_width" value="0.01"/>
+    <!-- === WORLD === -->
+    <link name="world_link"/>
+    <!-- === BASE === -->
+    <joint name="base_joint" type="fixed">
+        <parent link="world_link"/>
         <child link="base_link" />
-        <origin xyz="0.0 0.0 0.0" rpy="0 0 0"/>
+        <origin xyz="0 0 ${wheel_radius}" rpy="0 0 0"/>
     </joint>
     <link name="base_link">
         <visual>
-        <geometry>
-            <box size="${base_width} ${base_length} ${base_height}"/>
-        </geometry>
-        <origin xyz="0 0 0.25" rpy="0 0 0"/>
-        <material name="white">
-            <color rgba="1 1 1 1"/>
-        </material>
+            <geometry>
+                <box size="${base_length} ${base_width} ${base_height}"/>
+            </geometry>
+            <material name="white"/>
+            <origin xyz="0 0 0" rpy="0 0 0"/>
         </visual>
         <collision>
             <geometry>
-                <box size="${base_width} ${base_length} ${base_height}"/>
+                <box size="${base_length} ${base_width} ${base_height}"/>
             </geometry>
-            <origin xyz="0 0 25" rpy="0 0 0"/>
+            <origin xyz="0 0 0" rpy="0 0 0"/>
         </collision>
-        <xacro:box_inertia m="40.0" w="${base_width}" d="${base_length}" h="${base_height}"/>
+        <xacro:box_inertia m="1" l="${base_length}" w="${base_width}"  h="${base_height}">
+            <origin xyz="0 0 0" rpy="0 0 0"/>
+        </xacro:box_inertia>
     </link>
+    <!-- === WHEELS === -->
     <!-- <joint name="left_wheel_joint" type="continuous">
+        <parent link="base_link"/>
+        <child link="left_wheel_link" />
+        <origin xyz="0 ${base_width/2 + wheel_width/2 + 0.01} 0" rpy="-${pi/2} 0 0"/>
+        <axis xyz="0 0 1"/>
     </joint>
     <link name="left_wheel_link">
-    </link>
-    <link name="right_wheel_link">
+        <visual>
+            <geometry>
+                <cylinder radius="${wheel_radius}" length="${wheel_width}"/>
+            </geometry>
+            <material name="white"/>
+            <origin xyz="0 0 0" rpy="0 0 0"/>
+        </visual>
+        <collision>
+            <geometry>
+                <cylinder radius="${wheel_radius}" length="${wheel_width}"/>
+            </geometry>
+            <origin xyz="0 0 0" rpy="0 0 0"/>
+        </collision>
+        <xacro:cylinder_inertia m="1" r="${wheel_radius}" l="${wheel_width}">
+            <origin xyz="0 0 0" rpy="${pi/2} 0 0"/>
+        </xacro:cylinder_inertia>
     </link> -->
 </robot>

Commit message: feat: add URDF description for left and right wheels

File: twr_description/urdf/twr.urdf.xacro (robot description, xacro)
@@ -6,6 +6,6 @@
     <xacro:property name="base_width" value="0.4"/>
     <xacro:property name="base_height" value="0.1"/>
-    <xacro:property name="wheel_radius" value="0.2"/>
-    <xacro:property name="wheel_width" value="0.01"/>
+    <xacro:property name="wheel_radius" value="0.1"/>
+    <xacro:property name="wheel_width" value="0.05"/>
     <!-- === WORLD === -->
     <link name="world_link"/>
@@ -35,5 +35,5 @@
     </link>
     <!-- === WHEELS === -->
-    <!-- <joint name="left_wheel_joint" type="continuous">
+    <joint name="left_wheel_joint" type="continuous">
         <parent link="base_link"/>
         <child link="left_wheel_link" />
@@ -56,6 +56,30 @@
         </collision>
         <xacro:cylinder_inertia m="1" r="${wheel_radius}" l="${wheel_width}">
+            <origin xyz="0 0 0" rpy="-${pi/2} 0 0"/>
+        </xacro:cylinder_inertia>
+    </link>
+    <joint name="right_wheel_joint" type="continuous">
+        <parent link="base_link"/>
+        <child link="right_wheel_link" />
+        <origin xyz="0 -${base_width/2 + wheel_width/2 + 0.01} 0" rpy="${pi/2} 0 0"/>
+        <axis xyz="0 0 1"/>
+    </joint>
+    <link name="right_wheel_link">
+        <visual>
+            <geometry>
+                <cylinder radius="${wheel_radius}" length="${wheel_width}"/>
+            </geometry>
+            <material name="white"/>
+            <origin xyz="0 0 0" rpy="0 0 0"/>
+        </visual>
+        <collision>
+            <geometry>
+                <cylinder radius="${wheel_radius}" length="${wheel_width}"/>
+            </geometry>
+            <origin xyz="0 0 0" rpy="0 0 0"/>
+        </collision>
+        <xacro:cylinder_inertia m="1" r="${wheel_radius}" l="${wheel_width}">
             <origin xyz="0 0 0" rpy="${pi/2} 0 0"/>
         </xacro:cylinder_inertia>
-    </link> -->
+    </link>
 </robot>

Commit message: feat: add launch file for gazebo

File: twr_description/urdf/twr.urdf.xacro (robot description, xacro)
@@ -1,19 +1,24 @@
 <?xml version="1.0"?>
 <robot name="twr" xmlns:xacro="http://ros.org/wiki/xacro">
-    <xacro:include filename="inertia.macro.xacro"/>
-    <xacro:include filename="colors.xacro"/>
-    <xacro:property name="base_length" value="0.4"/>
-    <xacro:property name="base_width" value="0.4"/>
-    <xacro:property name="base_height" value="0.1"/>
-    <xacro:property name="wheel_radius" value="0.1"/>
-    <xacro:property name="wheel_width" value="0.05"/>
-    <xacro:property name="caster_wheel_radius" value="${wheel_radius/2-base_height/4}"/>
+    <xacro:include filename="_inertia.macro.xacro"/>
+    <xacro:include filename="_colors.xacro"/>
+    <xacro:property name="mm2m" value="0.001"/>
+    <xacro:property name="base_length" value="${200*mm2m}"/>
+    <xacro:property name="base_width" value="${200*mm2m}"/>
+    <xacro:property name="base_height" value="${40*mm2m}"/>
+    <xacro:property name="wheel_radius" value="${50*mm2m}"/>
+    <xacro:property name="wheel_width" value="${20*mm2m}"/>
+    <xacro:property name="caster_wheel_radius" value="${10*mm2m}"/>
+    <!-- ============= -->
     <!-- === WORLD === -->
+    <!-- ============= -->
     <link name="world_link"/>
+    <!-- ============ -->
     <!-- === BASE === -->
+    <!-- ============ -->
     <joint name="base_joint" type="fixed">
         <parent link="world_link"/>
         <child link="base_link" />
-        <origin xyz="0 0 ${wheel_radius}" rpy="0 0 0"/>
+        <origin xyz="0 0 ${wheel_radius+0.01}" rpy="0 0 0"/>
     </joint>
     <link name="base_link">
@@ -36,13 +41,15 @@
     </link>
     <!-- === CHASSIS === -->
-    <joint name="chassis_joint" type="fixed">
+    <!-- <joint name="chassis_joint" type="fixed">
         <parent link="base_link"/>
         <child link="chassis_link" />
         <origin xyz="0 0 0" rpy="0 0 0"/>
     </joint>
-    <link name="chassis_link"></link>
+    <link name="chassis_link"></link> -->
+    <!-- ============== -->
     <!-- === WHEELS === -->
+    <!-- ============== -->
     <joint name="left_wheel_joint" type="continuous">
-        <parent link="chassis_link"/>
+        <parent link="base_link"/>
         <child link="left_wheel_link" />
         <origin xyz="0 ${base_width/2 + wheel_width/2 + 0.01} 0" rpy="-${pi/2} 0 0"/>
@@ -68,5 +75,5 @@
     </link>
     <joint name="right_wheel_joint" type="continuous">
-        <parent link="chassis_link"/>
+        <parent link="base_link"/>
         <child link="right_wheel_link" />
         <origin xyz="0 -${base_width/2 + wheel_width/2 + 0.01} 0" rpy="${pi/2} 0 0"/>
@@ -91,9 +98,11 @@
         </xacro:cylinder_inertia>
     </link>
+    <!-- ===================== -->
     <!-- === CASTER WHEELS === -->
+    <!-- ===================== -->
     <joint name="caster_front_wheel_joint" type="continuous">
         <parent link="base_link"/>
         <child link="caster_front_wheel_link"/>
-        <origin xyz="${base_length/2-caster_wheel_radius} 0 -${base_height/2+caster_wheel_radius+0.01}" rpy="0 0 0"/>
+        <origin xyz="${base_length/2-caster_wheel_radius} 0 -${wheel_radius-caster_wheel_radius-1*mm2m}" rpy="0 0 0"/>
         <axis xyz="1 1 1"/>
     </joint>
@@ -108,9 +117,9 @@
         <collision>
             <geometry>
-                <sphere radius="${wheel_radius}"/>
+                <sphere radius="${caster_wheel_radius}"/>
             </geometry>
             <origin xyz="0 0 0" rpy="0 0 0"/>
         </collision>
-        <xacro:sphere_inertia m="0.1" r="${wheel_radius}">
+        <xacro:sphere_inertia m="0.01" r="${caster_wheel_radius}">
             <origin xyz="0 0 0" rpy="0 0 0"/>
         </xacro:sphere_inertia>
@@ -119,5 +128,5 @@
         <parent link="base_link"/>
         <child link="caster_back_wheel_link"/>
-        <origin xyz="-${base_length/2-caster_wheel_radius} 0 -${base_height/2+caster_wheel_radius+0.01}" rpy="0 0 0"/>
+        <origin xyz="-${base_length/2-caster_wheel_radius} 0 -${wheel_radius-caster_wheel_radius-1*mm2m}" rpy="0 0 0"/>
         <axis xyz="1 1 1"/>
     </joint>
@@ -132,9 +141,9 @@
         <collision>
             <geometry>
-                <sphere radius="${wheel_radius}"/>
+                <sphere radius="${caster_wheel_radius}"/>
             </geometry>
             <origin xyz="0 0 0" rpy="0 0 0"/>
         </collision>
-        <xacro:sphere_inertia m="0.1" r="${wheel_radius}">
+        <xacro:sphere_inertia m="0.01" r="${caster_wheel_radius}">
             <origin xyz="0 0 0" rpy="0 0 0"/>
         </xacro:sphere_inertia>
